File: makita_protector/makita_protector.kicad_pcb (KiCad board)
At the start: 2 copper layers, 48 x 55 mm, 64 parts, among them J1 12V, J2 GND, J3 FORCE_ON, J4 GND, J5 FORCE_OFF, J6 GND, Q1 SQJ457EP, Q2 BSS123, U1 TPS54302, U2 LM2903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

Commit message: updated layput
Parts:
- H1, H2, H3, H4: footprint MountingHole:MountingHole_3.2mm_M3_DIN965_Pad -> MountingHole:MountingHole_3.2mm_M3_DIN965
- moved R2 3.49 mm to (148.6, 79.0)
- moved R1 3.06 mm to (147.0, 82.6)
Routing:
- net +12V: track 65.5 -> 105.3 mm, vias 0 -> 2
- net VBUS: track 51.8 -> 17.2 mm
- net Net-(J5-Pad1): track 0.00 -> 25.6 mm
- net Net-(R10-Pad2): track 0.00 -> 22.1 mm, vias 0 -> 2
- net Net-(C5-Pad1): track 1.96 -> 17.8 mm
- net Net-(R10-Pad1): track 0.00 -> 12.3 mm
- net Net-(C3-Pad2): track 0.00 -> 9.99 mm
- net GND: track 0.00 -> 9.08 mm
- net Net-(C13-Pad1): track 0.00 -> 9.02 mm, vias 0 -> 2
- net Net-(C8-Pad1): track 0.00 -> 6.92 mm
- net Net-(R1-Pad2): track 0.00 -> 6.33 mm
- net Net-(C6-Pad2): track 0.00 -> 6.15 mm
- net Net-(C16-Pad2): track 0.00 -> 6.15 mm
- net Net-(R11-Pad2): track 0.00 -> 5.94 mm
- net Net-(Q2-Pad3): track 0.00 -> 5.51 mm
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- added copper zone on F.Cu, net +12V
- added copper zone on B.Cu, net GND
- added copper zone on F.Cu, net GND
- added copper zone on B.Cu, net Net-(C4-Pad1)
- added copper zone on F.Cu, net Net-(C4-Pad1)
- added copper zone on F.Cu, net VBUS

Commit message: updated layput
Routing:
- net VBUS: track 17.2 -> 33.0 mm, vias 0 -> 4

Commit message: updated layput
Parts:
- moved R12 3.49 mm to (162.4, 79.1)
- moved R11 3.06 mm to (160.8, 82.7)
Routing:
- net VBUS: track 33.0 -> 83.5 mm
- net +12V: track 105.3 -> 118.6 mm, vias 2 -> 4
- net GND: track 9.08 -> 18.2 mm, vias 0 -> 26
- net Net-(C13-Pad1): track 9.02 -> 12.0 mm
- net Net-(C3-Pad1): track 0.00 -> 1.69 mm
- net Net-(D1-Pad1): track 0.00 -> 1.56 mm
- net Net-(C14-Pad1): track 4.09 -> 4.27 mm, vias 0 -> 17
- net (no net): vias 0 -> 1
- added copper zone on B.Cu, net Net-(C14-Pad1)
- added copper zone on F.Cu, net Net-(C14-Pad1)

Commit message: final version for production v1
Parts:
- added FID1: Fiducial, makita_protector:Fiducial_1mm_Mask2mm_Paste, F.Cu at (129.8, 58.4)
- added FID2: Fiducial, makita_protector:Fiducial_1mm_Mask2mm_Paste, F.Cu at (169.9, 58.9)
- added FID3: Fiducial, makita_protector:Fiducial_1mm_Mask2mm_Paste, F.Cu at (164.1, 99.3)
- added LOGO1: oshw, Symbol:OSHW-Logo2_7.3x6mm_SilkScreen, F.Cu at (143.0, 105.9)
- added LOGO2: Kicad, Symbol:KiCad-Logo2_5mm_SilkScreen, F.Cu at (161.0, 105.7)
- moved J1 15.0 mm to (148.8, 106.2)
- moved J4 12.1 mm to (140.0, 70.1)
- moved C10 5.37 mm to (158.2, 58.7), turned to 90 degrees
- moved J2 3.51 mm to (140.0, 73.9)
- moved J6 3.17 mm to (136.7, 72.1)
- moved J3 2.19 mm to (136.7, 65.3)
- moved R14 2.04 mm to (160.5, 58.7)
- moved J5 0.94 mm to (136.7, 58.7)
- turned D4 to 180 degrees
Routing:
- net +12V: track 118.6 -> 92.4 mm
- net Net-(R14-Pad2): track 3.20 -> 5.61 mm
- net Net-(C13-Pad1): track 12.0 -> 13.3 mm
- net Net-(J5-Pad1): track 25.6 -> 24.3 mm
- net VBUS: track 83.5 -> 84.4 mm
- net Net-(C3-Pad2): track 9.99 -> 10.9 mm
- net GND: vias 26 -> 64
Other:
- board text added: "GND"
- board text added: "OFF"
- board text added: "ON"
- board text added: "v1 MBP 01/2020"

Commit message: updated values after initial testing
Parts:
- C3: value 100n -> 0R
- R10: value 1Meg -> 10k
- R15: value 100k -> 33k
- R16: value 33k -> 1k
- R20, R21: value 100k -> 10k
